File: Schematic and Preliminary Layout/Distance sensor PSC.kicad_sch (KiCad schematic)
At the start: 12 parts, among them U1 HC-SR04

Commit message: Updated Schematic
Parts:
- U1: symbol HC-SR04:HC-SR04 -> Distance sensor:HC-SR04
- U2: symbol Oled_SSD1306_6pin:SSD1306_6-pin -> OLED Display:SSD1306_6-pin
Connections:
- net +5V renamed 5V_USB
- net 5V_USB: no longer BT1.1 (+)
- new net 5V_BAT: BT1.1 (+)
