File: Schematic and Preliminary Layout/Distance sensor PSC.kicad_pcb (KiCad board)
At the start: 2 copper layers, 87 x 84.5 mm, 15 parts, among them U1 HC-SR04

Commit message: Updated PCB
Parts:
- moved D1 0.50 mm to (153.0, 110.0)
- moved D2 0.50 mm to (145.2, 110.0)
- moved D3 0.50 mm to (137.5, 110.0)
- moved U2 0.50 mm to (152.9, 80.0)
Routing:
- net Net-(D3-A): track 11.4 -> 10.9 mm
- net Net-(D2-A): track 17.8 -> 17.3 mm
- net Net-(D1-A): track 25.5 -> 25.0 mm
- net Net-(A1-SDA/IO23): track 39.8 -> 39.3 mm
- net +3.3V: track 59.2 -> 59.7 mm
- net GND: vias 1 -> 9
Changed lines of the file:
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@@
 	(footprint "LED_THT:LED_D5.0mm"
 		(layer "B.Cu")
-		(at 137.5 109.5 180)
+		(at 137.5 110 180)
 		(descr "LED, diameter 5.0mm, 2 pins, http://cdn-reichelt.de/documents/datenblatt/A500/LL-504BC2E-009.pdf, generated by kicad-footprint-generator")
 		(tags "LED")
@@
 	(footprint "Display:Adafruit_SSD1306"
 		(layer "B.Cu")
-		(at 152.912 79.5 180)
+		(at 152.912 80 180)
 		(descr "Adafruit SSD1306 OLED 1.3 inch 128x64 I2C & SPI https://learn.adafruit.com/monochrome-oled-breakouts/downloads")
 		(tags "Adafruit SSD1306 OLED 1.3 inch 128x64 I2C & SPI ")
@@
 	(footprint "LED_THT:LED_D5.0mm"
 		(layer "B.Cu")
-		(at 153 109.5 180)
+		(at 153 110 180)
 		(descr "LED, diameter 5.0mm, 2 pins, http://cdn-reichelt.de/documents/datenblatt/A500/LL-504BC2E-009.pdf, generated by kicad-footprint-generator")
 		(tags "LED")
@@
 	(footprint "LED_THT:LED_D5.0mm"
 		(layer "B.Cu")
-		(at 145.25 109.5 180)
+		(at 145.25 110 180)
 		(descr "LED, diameter 5.0mm, 2 pins, http://cdn-reichelt.de/documents/datenblatt/A500/LL-504BC2E-009.pdf, generated by kicad-footprint-generator")
 		(tags "LED")
@@
 	)
 	(segment
+		(start 151.211 77.799)
+		(end 151.211 78.299)
+		(width 0.7)
+		(layer "F.Cu")
+		(net 15)
+	)
+	(segment
 		(start 126.701 77.799)
 		(end 126.5 78)
@@
 	)
 	(segment
-		(start 152.912 79.5)
-		(end 151.211 77.799)
+		(start 151.211 78.299)
+		(end 152.912 80)
 		(width 0.7)
 		(layer "F.Cu")
@@
 	)
 	(segment
-		(start 140.212 79.5)
-		(end 140.212 85.728)
+		(start 140.212 85.728)
+		(end 140.212 80)
 		(width 0.4)
 		(layer "F.Cu")
@@
 	)
 	(segment
-		(start 139.73524 78.349)
-		(end 138.823 79.26124)
+		(start 141.501 78.749)
+		(end 142.752 80)
 		(width 0.4)
 		(layer "F.Cu")
@@
 	)
 	(segment
-		(start 142.752 79.5)
-		(end 141.601 78.349)
+		(start 138.961 79.481818)
+		(end 139.693818 78.749)
 		(width 0.4)
 		(layer "F.Cu")
@@
 	)
 	(segment
-		(start 138.823 84.577)
-		(end 116.5 106.9)
+		(start 138.961 84.439)
+		(end 138.961 79.481818)
 		(width 0.4)
 		(layer "F.Cu")
@@
 	)
 	(segment
-		(start 141.601 78.349)
-		(end 139.73524 78.349)
+		(start 139.693818 78.749)
+		(end 141.501 78.749)
 		(width 0.4)
 		(layer "F.Cu")
@@
 	)
 	(segment
-		(start 138.823 79.26124)
-		(end 138.823 84.577)
+		(start 116.5 106.9)
+		(end 138.961 84.439)
 		(width 0.4)
 		(layer "F.Cu")
 		(net 24)
+	)
+	(via
+		(at 140 115)
+		(size 0.6)
+		(drill 0.3)
+		(layers "F.Cu" "B.Cu")
+		(free yes)
+		(net 26)
+	)
+	(via
+		(at 132 59)
+		(size 0.6)
+		(drill 0.3)
+		(layers "F.Cu" "B.Cu")
+		(free yes)
+		(net 26)
+	)
+	(via
+		(at 114.5 61)
+		(size 0.6)
+		(drill 0.3)
+		(layers "F.Cu" "B.Cu")
+		(free yes)
+		(net 26)
+	)
+	(via
+		(at 156 116)
+		(size 0.6)
+		(drill 0.3)
+		(layers "F.Cu" "B.Cu")
+		(free yes)
+		(net 26)
+	)
+	(via
+		(at 137.5 70.5)
+		(size 0.6)
+		(drill 0.3)
+		(layers "F.Cu" "B.Cu")
+		(free yes)
+		(net 26)
+	)
+	(via
+		(at 151.5 75.5)
+		(size 0.6)
+		(drill 0.3)
+		(layers "F.Cu" "B.Cu")
+		(free yes)
+		(net 26)
+	)
+	(via
+		(at 147 115.5)
+		(size 0.6)
+		(drill 0.3)
+		(layers "F.Cu" "B.Cu")
+		(free yes)
+		(net 26)
 	)
 	(via
@@
 		(net 26)
 	)
+	(via
+		(at 92.5 79)
+		(size 0.6)
+		(drill 0.3)
+		(layers "F.Cu" "B.Cu")
+		(free yes)
+		(net 26)
+	)
 	(segment
 		(start 141.809 74.651)
@@
 	(segment
 		(start 150.46 115.29)
-		(end 150.46 109.5)
+		(end 150.46 110)
 		(width 0.4)
 		(layer "F.Cu")
 		(net 28)
+	)
+	(segment
+		(start 142.71 118.6)
+		(end 142.71 110)
+		(width 0.4)
+		(layer "F.Cu")
+		(net 29)
 	)
 	(segment
@@
 	)
 	(segment
-		(start 142.71 118.6)
-		(end 142.71 109.5)
-		(width 0.4)
-		(layer "F.Cu")
-		(net 29)
-	)
-	(segment
 		(start 136.56 118.06)
 		(end 134.96 116.46)
@@
 	(segment
 		(start 134.96 116.46)
-		(end 134.96 109.5)
-		(width 0.4)
-		(layer "F.Cu")
+		(end 134.96 110)
+		(width 0.4)
+		(layer "F.Cu")

Commit message: added team version and date to PCB
Other:
- board text added: "Team 15 Rev: 3.0 11-20-2025"
Changed lines of the file:
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@@
 		(layer "Edge.Cuts")
+	)
+	(gr_text "Team 15\nRev: 3.0\n11-20-2025\n"
+		(at 154.5 57.5 0)
+		(layer "F.Cu")
+		(effects
+			(font
+				(size 1.5 1.5)
+				(thickness 0.3)
+				(bold yes)
+			)
+			(justify left bottom)
+		)
 	)
 	(gr_text "Yellow"
